File: navrh vzorku/ESP32/ESP32.sch (EAGLE design)
At the start: 16 parts, among them U1 ESP-WROOM-32

Commit message: Funkcni vzorky eagle
Parts:
- added LED1: (no value), led:LED5MM
- added R7: 650, rcl:R-EU_0207/10
- added SG1: F/CM12P, buzzer:F/CM12P
Connections:
- removed net N$9: R5.2, R6.2, U1.GND@15, UARTMODE.2
- new net N$13: SG1.1, U1.IO14
- new net N$14: LED1.C, U1.IO12
- new net N$15: LED1.A, R7.2
- new net N$16: R5.2, R6.2, SG1.2, U1.GND@15, UARTMODE.2
- net N$2: now also R7.1
Changed lines of the file:
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@@
 <layer number="97" name="Info" color="7" fill="1" visible="yes" active="yes"/>
 <layer number="98" name="Guide" color="6" fill="1" visible="yes" active="yes"/>
+<layer number="99" name="SpiceOrder" color="5" fill="1" visible="yes" active="yes"/>
 </layers>
 <schematic xreflabel="%F%N/%S.%C%R" xrefpart="/%S.%C%R">
@@
 <part name="R5" library="rcl" library_urn="urn:adsk.eagle:library:334" deviceset="R-EU_" device="0207/10" package3d_urn="urn:adsk.eagle:package:23491/2" value="10k"/>
 <part name="R6" library="rcl" library_urn="urn:adsk.eagle:library:334" deviceset="R-EU_" device="0207/10" package3d_urn="urn:adsk.eagle:package:23491/2" value="10k"/>
+<part name="LED1" library="led" library_urn="urn:adsk.eagle:library:259" deviceset="LED" device="5MM" package3d_urn="urn:adsk.eagle:package:15799/2"/>
+<part name="R7" library="rcl" library_urn="urn:adsk.eagle:library:334" deviceset="R-EU_" device="0207/10" package3d_urn="urn:adsk.eagle:package:23491/2" value="650"/>
+<part name="SG1" library="buzzer" library_urn="urn:adsk.eagle:library:113" deviceset="F/CM12P" device="" package3d_urn="urn:adsk.eagle:package:5265/1"/>
 </parts>
 <sheets>
@@
 <attribute name="NAME" x="211.8614" y="34.29" size="1.778" layer="95" rot="R90"/>
 <attribute name="VALUE" x="214.122" y="34.29" size="1.778" layer="96" rot="R90"/>
+</instance>
+<instance part="LED1" gate="G$1" x="177.8" y="60.96" smashed="yes" rot="R180">
+<attribute name="NAME" x="174.244" y="62.992" size="1.778" layer="95" rot="R270"/>
+<attribute name="VALUE" x="172.085" y="65.532" size="1.778" layer="96" rot="R270"/>
+</instance>
+<instance part="R7" gate="G$1" x="177.8" y="50.8" smashed="yes" rot="R90">
+<attribute name="NAME" x="181.3814" y="46.99" size="1.778" layer="95" rot="R90"/>
+<attribute name="VALUE" x="183.642" y="46.99" size="1.778" layer="96" rot="R90"/>
+</instance>
+<instance part="SG1" gate="G$1" x="170.18" y="35.56" smashed="yes" rot="R180">
+<attribute name="NAME" x="172.72" y="29.21" size="1.778" layer="95" rot="R180"/>
+<attribute name="VALUE" x="163.83" y="35.56" size="1.778" layer="96" rot="R180"/>
 </instance>
 </instances>
@@
 <wire x1="233.68" y1="53.34" x2="233.68" y2="45.72" width="0.1524" layer="91"/>
 <wire x1="233.68" y1="45.72" x2="193.04" y2="45.72" width="0.1524" layer="91"/>
-<wire x1="193.04" y1="45.72" x2="162.56" y2="45.72" width="0.1524" layer="91"/>
+<wire x1="193.04" y1="45.72" x2="177.8" y2="45.72" width="0.1524" layer="91"/>
+<wire x1="177.8" y1="45.72" x2="162.56" y2="45.72" width="0.1524" layer="91"/>
 <wire x1="162.56" y1="45.72" x2="162.56" y2="99.06" width="0.1524" layer="91"/>
 <junction x="162.56" y="99.06"/>
@@
 <wire x1="193.04" y1="33.02" x2="193.04" y2="20.32" width="0.1524" layer="91"/>
 <junction x="193.04" y="33.02"/>
+<pinref part="R7" gate="G$1" pin="1"/>
+<junction x="177.8" y="45.72"/>
 </segment>
 </net>
@@
 </segment>
 </net>
-<net name="N$9" class="0">
-<segment>
+<net name="N$10" class="0">
+<segment>
+<pinref part="R4" gate="G$1" pin="2"/>
+<wire x1="109.22" y1="114.3" x2="109.22" y2="119.38" width="0.1524" layer="91"/>
+<pinref part="NAPAJENI" gate="G$1" pin="2"/>
+<wire x1="109.22" y1="119.38" x2="114.3" y2="119.38" width="0.1524" layer="91"/>
+<wire x1="109.22" y1="114.3" x2="121.92" y2="114.3" width="0.1524" layer="91"/>
+<junction x="109.22" y="114.3"/>
+<pinref part="MERENI_UBYTKU_NAPETI" gate="G$1" pin="1"/>
+</segment>
+</net>
+<net name="N$11" class="0">
+<segment>
+<pinref part="U1" gate="G$1" pin="IO2"/>
+<pinref part="S2" gate="1" pin="S"/>
+<wire x1="215.9" y1="58.42" x2="215.9" y2="20.32" width="0.1524" layer="91"/>
+<wire x1="215.9" y1="20.32" x2="210.82" y2="20.32" width="0.1524" layer="91"/>
+<pinref part="R5" gate="G$1" pin="1"/>
+<wire x1="210.82" y1="20.32" x2="205.74" y2="20.32" width="0.1524" layer="91"/>
+<junction x="210.82" y="20.32"/>
+</segment>
+</net>
+<net name="N$12" class="0">
+<segment>
+<pinref part="S1" gate="1" pin="S"/>
+<wire x1="205.74" y1="33.02" x2="208.28" y2="33.02" width="0.1524" layer="91"/>
+<pinref part="U1" gate="G$1" pin="IO15"/>
+<wire x1="208.28" y1="33.02" x2="213.36" y2="33.02" width="0.1524" layer="91"/>
+<wire x1="213.36" y1="33.02" x2="213.36" y2="58.42" width="0.1524" layer="91"/>
+<pinref part="R6" gate="G$1" pin="1"/>
+<junction x="208.28" y="33.02"/>
+</segment>
+</net>
+<net name="N$13" class="0">
+<segment>
+<pinref part="U1" gate="G$1" pin="IO14"/>
+<wire x1="180.34" y1="71.12" x2="172.72" y2="71.12" width="0.1524" layer="91"/>
+<pinref part="SG1" gate="G$1" pin="1"/>
+<wire x1="172.72" y1="38.1" x2="172.72" y2="71.12" width="0.1524" layer="91"/>
+</segment>
+</net>
+<net name="N$14" class="0">
+<segment>
+<pinref part="U1" gate="G$1" pin="IO12"/>
+<pinref part="LED1" gate="G$1" pin="C"/>
+<wire x1="180.34" y1="68.58" x2="177.8" y2="68.58" width="0.1524" layer="91"/>
+<wire x1="177.8" y1="68.58" x2="177.8" y2="66.04" width="0.1524" layer="91"/>
+</segment>
+</net>
+<net name="N$15" class="0">
+<segment>
+<pinref part="R7" gate="G$1" pin="2"/>
+<pinref part="LED1" gate="G$1" pin="A"/>
+<wire x1="177.8" y1="58.42" x2="177.8" y2="55.88" width="0.1524" layer="91"/>
+</segment>
+</net>
+<net name="N$16" class="0">
+<segment>
+<pinref part="SG1" gate="G$1" pin="2"/>
+<wire x1="165.1" y1="38.1" x2="165.1" y2="40.64" width="0.1524" layer="91"/>
+<wire x1="165.1" y1="40.64" x2="187.96" y2="40.64" width="0.1524" layer="91"/>
+<wire x1="187.96" y1="40.64" x2="187.96" y2="53.34" width="0.1524" layer="91"/>
 <pinref part="UARTMODE" gate="G$1" pin="2"/>
 <wire x1="243.84" y1="66.04" x2="228.6" y2="66.04" width="0.1524" layer="91"/>
@@
 <wire x1="210.82" y1="50.8" x2="208.28" y2="50.8" width="0.1524" layer="91"/>
 <wire x1="208.28" y1="50.8" x2="193.04" y2="50.8" width="0.1524" layer="91"/>
-<wire x1="193.04" y1="50.8" x2="193.04" y2="58.42" width="0.1524" layer="91"/>
+<wire x1="193.04" y1="50.8" x2="193.04" y2="53.34" width="0.1524" layer="91"/>
 <pinref part="R5" gate="G$1" pin="2"/>
+<wire x1="193.04" y1="53.34" x2="193.04" y2="58.42" width="0.1524" layer="91"/>
 <wire x1="210.82" y1="30.48" x2="210.82" y2="50.8" width="0.1524" layer="91"/>
 <junction x="210.82" y="50.8"/>
@@
 <wire x1="208.28" y1="43.18" x2="208.28" y2="50.8" width="0.1524" layer="91"/>
 <junction x="208.28" y="50.8"/>
-</segment>
-</net>
-<net name="N$10" class="0">
-<segment>
-<pinref part="R4" gate="G$1" pin="2"/>
-<wire x1="109.22" y1="114.3" x2="109.22" y2="119.38" width="0.1524" layer="91"/>
-<pinref part="NAPAJENI" gate="G$1" pin="2"/>
-<wire x1="109.22" y1="119.38" x2="114.3" y2="119.38" width="0.1524" layer="91"/>
-<wire x1="109.22" y1="114.3" x2="121.92" y2="114.3" width="0.1524" layer="91"/>
-<junction x="109.22" y="114.3"/>
-<pinref part="MERENI_UBYTKU_NAPETI" gate="G$1" pin="1"/>
-</segment>
-</net>
-<net name="N$11" class="0">
-<segment>
-<pinref part="U1" gate="G$1" pin="IO2"/>
-<pinref part="S2" gate="1" pin="S"/>
-<wire x1="215.9" y1="58.42" x2="215.9" y2="20.32" width="0.1524" layer="91"/>
-<wire x1="215.9" y1="20.32" x2="210.82" y2="20.32" width="0.1524" layer="91"/>
-<pinref part="R5" gate="G$1" pin="1"/>
-<wire x1="210.82" y1="20.32" x2="205.74" y2="20.32" width="0.1524" layer="91"/>
-<junction x="210.82" y="20.32"/>
-</segment>
-</net>
-<net name="N$12" class="0">
-<segment>
-<pinref part="S1" gate="1" pin="S"/>
-<wire x1="205.74" y1="33.02" x2="208.28" y2="33.02" width="0.1524" layer="91"/>
-<pinref part="U1" gate="G$1" pin="IO15"/>
-<wire x1="208.28" y1="33.02" x2="213.36" y2="33.02" width="0.1524" layer="91"/>
-<wire x1="213.36" y1="33.02" x2="213.36" y2="58.42" width="0.1524" layer="91"/>
-<pinref part="R6" gate="G$1" pin="1"/>
-<junction x="208.28" y="33.02"/>
-</segment>
-</net>
+<wire x1="187.96" y1="53.34" x2="193.04" y2="53.34" width="0.1524" layer="91"/>
+<junction x="193.04" y="53.34"/>
+</segment>
+</net>

Commit message: Program funčního vzorku ESP
Parts:
- added S3: (no value), switch-omron:10-XX
- R7: value 650 -> 100k
Connections:
- removed net N$15: LED1.A, R7.2
- new net N$9: R7.2, U1.IO12
- net N$14: now also LED1.A, R7.1; no longer LED1.C, U1.IO12
- net N$16: now also LED1.C
- net N$2: no longer R7.1
- net N$3: now also S3.P1
- net N$5: now also S3.S1
Other:
- moved on the sheet: LED1, R2, R7, SG1

Commit message: funkcni vzorek ESP8266
Connections:
- net N$3: now also S3.P; no longer S3.P1
- net N$5: now also S3.S; no longer S3.S1
Changed lines of the file:
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@@
 <wire x1="106.68" y1="101.6" x2="165.1" y2="101.6" width="0.1524" layer="91"/>
 <junction x="106.68" y="101.6"/>
-<pinref part="S3" gate="1" pin="P1"/>
+<pinref part="S3" gate="1" pin="P"/>
 <wire x1="165.1" y1="101.6" x2="180.34" y2="101.6" width="0.1524" layer="91"/>
-<wire x1="165.1" y1="101.6" x2="165.1" y2="109.22" width="0.1524" layer="91"/>
+<wire x1="165.1" y1="101.6" x2="165.1" y2="111.76" width="0.1524" layer="91"/>
 <junction x="165.1" y="101.6"/>
 </segment>
@@
 <net name="N$5" class="0">
 <segment>
-<pinref part="S3" gate="1" pin="S1"/>
-<wire x1="175.26" y1="109.22" x2="175.26" y2="96.52" width="0.1524" layer="91"/>
+<pinref part="S3" gate="1" pin="S"/>
+<wire x1="175.26" y1="111.76" x2="175.26" y2="96.52" width="0.1524" layer="91"/>
 <pinref part="U1" gate="G$1" pin="EN"/>
 <wire x1="175.26" y1="96.52" x2="180.34" y2="96.52" width="0.1524" layer="91"/>

Commit message: Plosne spoje
Parts:
- R7: value 100k -> 10
Connections:
- removed net N$16: LED1.C, R5.2, R6.2, SG1.2, U1.GND@15, UARTMODE.2
- removed net N$3: C1.2, C2.2, NAPAJENI.1, S3.P, U$1.GND, U1.GND@1
- new net GND: C1.2, C2.2, LED1.C, NAPAJENI.1, R5.2, R6.2, S3.P, S3.P1, SG1.2, U$1.GND, U1.GND@1, U1.GND@15, UARTMODE.2
- net N$5: now also S3.S1

Commit message: Finalni verze
Parts:
- removed MERENI_UBYTKU_NAPETI: (no value), pinhead:PINHD-1X2
- removed R1: 100k, rcl:R-EU_0207/10
- removed R4: 10, rcl:R-EU_0207/10
- removed U$1: LDLN030, WT8266:LDLN030
- added C3: 0.1u, capacitor-wima:C2.5/2
- added D1, D2: 1N4004, diode:1N4004
- added JP1: (no value), pinhead:PINHD-1X3
- added JP2, JP3: (no value), pinhead:PINHD-1X2
- added R8: (no value), rcl:R-EU_0207/10
- C1, C2: value (none) -> 22u
Connections:
- removed net N$10: MERENI_UBYTKU_NAPETI.1, NAPAJENI.2, R4.2
- removed net N$4: R1.1, U$1.PG
- removed net N$9: R7.2, U1.IO12
- new net N$15: D1.C, D2.C, JP1.1, R8.2, U1.IO32
- new net N$17: D1.A, JP2.1
- new net N$18: D2.A, JP3.2
- new net N$3: JP1.3, R2.2, S3.S, S3.S1
- net GND: now also C3.2, R8.1; no longer U$1.GND
- net N$1: now also SG1.1, U1.IO18; no longer C1.1, MERENI_UBYTKU_NAPETI.2, R4.1, U$1.EN, U$1.IN
- net N$11: now also JP2.2
- net N$12: now also JP3.1
- net N$13: now also R7.2; no longer SG1.1
- net N$2: now also C1.1, C3.1, NAPAJENI.2; no longer R1.2, U$1.OUT
- net N$5: now also JP1.2; no longer R2.2, S3.S, S3.S1
Other:
- moved on the sheet: C1, C2, LED1, NAPAJENI, R2, R5, R7, S1, S2, S3, SG1
