File: navrh vzorku/ESP8266/esp8266.sch (EAGLE design)
At the start: 23 parts

Commit message: funkcni vzorek ESP8266
Connections:
- net N$13: now also S1.S1; no longer S1.S
- net N$15: now also R8.1; no longer LED1.C
- net N$16: now also R8.2; no longer R8.1
- net N$18: now also LED1.C
- net N$2: no longer R8.2
- net N$6: now also S2.P1; no longer S2.P
Other:
- moved on the sheet: LED1, R8
Changed lines of the file:
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@@
 <attribute name="VALUE" x="125.73" y="23.622" size="1.778" layer="96" rot="R180"/>
 </instance>
-<instance part="LED1" gate="G$1" x="68.58" y="30.48" smashed="yes" rot="R90">
-<attribute name="NAME" x="73.152" y="34.036" size="1.778" layer="95" rot="R180"/>
-<attribute name="VALUE" x="73.152" y="36.195" size="1.778" layer="96" rot="R180"/>
-</instance>
-<instance part="R8" gate="G$1" x="55.88" y="30.48" smashed="yes" rot="R180">
-<attribute name="NAME" x="57.15" y="34.0614" size="1.778" layer="95" rot="R180"/>
-<attribute name="VALUE" x="57.15" y="36.322" size="1.778" layer="96" rot="R180"/>
+<instance part="LED1" gate="G$1" x="60.96" y="30.48" smashed="yes" rot="R270">
+<attribute name="NAME" x="56.388" y="26.924" size="1.778" layer="95"/>
+<attribute name="VALUE" x="56.388" y="24.765" size="1.778" layer="96"/>
+</instance>
+<instance part="R8" gate="G$1" x="68.58" y="30.48" smashed="yes" rot="R180">
+<attribute name="NAME" x="69.85" y="34.0614" size="1.778" layer="95" rot="R180"/>
+<attribute name="VALUE" x="69.85" y="36.322" size="1.778" layer="96" rot="R180"/>
 </instance>
 <instance part="SG1" gate="G$1" x="76.2" y="12.7" smashed="yes" rot="R180">
@@
 <junction x="99.06" y="63.5"/>
 <wire x1="111.76" y1="63.5" x2="111.76" y2="60.96" width="0.1524" layer="91"/>
-<pinref part="S2" gate="1" pin="P"/>
+<pinref part="S2" gate="1" pin="P1"/>
 <wire x1="111.76" y1="60.96" x2="111.76" y2="45.72" width="0.1524" layer="91"/>
-<wire x1="111.76" y1="45.72" x2="114.3" y2="45.72" width="0.1524" layer="91"/>
+<wire x1="111.76" y1="45.72" x2="114.3" y2="43.18" width="0.1524" layer="91"/>
 <pinref part="S1" gate="1" pin="P"/>
 <wire x1="114.3" y1="60.96" x2="111.76" y2="60.96" width="0.1524" layer="91"/>
@@
 <segment>
 <pinref part="R5" gate="G$1" pin="2"/>
-<pinref part="S1" gate="1" pin="S"/>
+<pinref part="S1" gate="1" pin="S1"/>
 <pinref part="U$1" gate="G$1" pin="IO14"/>
-<wire x1="129.54" y1="60.96" x2="124.46" y2="60.96" width="0.1524" layer="91"/>
+<wire x1="129.54" y1="60.96" x2="124.46" y2="58.42" width="0.1524" layer="91"/>
 <wire x1="93.98" y1="60.96" x2="104.14" y2="60.96" width="0.1524" layer="91"/>
 <wire x1="104.14" y1="60.96" x2="104.14" y2="55.88" width="0.1524" layer="91"/>
@@
 <pinref part="C2" gate="G$1" pin="1"/>
 <pinref part="U$1" gate="G$1" pin="3.3V"/>
-<wire x1="38.1" y1="63.5" x2="48.26" y2="63.5" width="0.1524" layer="91"/>
+<wire x1="38.1" y1="63.5" x2="53.34" y2="63.5" width="0.1524" layer="91"/>
 <junction x="38.1" y="63.5"/>
 <pinref part="R2" gate="G$1" pin="2"/>
@@
 <wire x1="139.7" y1="25.4" x2="139.7" y2="45.72" width="0.1524" layer="91"/>
 <junction x="139.7" y="45.72"/>
-<wire x1="53.34" y1="63.5" x2="48.26" y2="63.5" width="0.1524" layer="91"/>
-<wire x1="48.26" y1="63.5" x2="48.26" y2="30.48" width="0.1524" layer="91"/>
-<wire x1="48.26" y1="30.48" x2="50.8" y2="30.48" width="0.1524" layer="91"/>
-<pinref part="R8" gate="G$1" pin="2"/>
 </segment>
 </net>
@@
 <net name="N$15" class="0">
 <segment>
-<pinref part="LED1" gate="G$1" pin="C"/>
-<wire x1="73.66" y1="30.48" x2="76.2" y2="30.48" width="0.1524" layer="91"/>
 <pinref part="U$1" gate="G$1" pin="IO13"/>
 <wire x1="76.2" y1="30.48" x2="76.2" y2="38.1" width="0.1524" layer="91"/>
+<pinref part="R8" gate="G$1" pin="1"/>
+<wire x1="73.66" y1="30.48" x2="76.2" y2="30.48" width="0.1524" layer="91"/>
 </segment>
 </net>
 <net name="N$16" class="0">
 <segment>
-<pinref part="R8" gate="G$1" pin="1"/>
 <pinref part="LED1" gate="G$1" pin="A"/>
-<wire x1="60.96" y1="30.48" x2="66.04" y2="30.48" width="0.1524" layer="91"/>
+<pinref part="R8" gate="G$1" pin="2"/>
 </segment>
 </net>
@@
 <segment>
 <pinref part="U$1" gate="G$1" pin="IO5"/>
+<pinref part="SG1" gate="G$1" pin="1"/>
 <wire x1="78.74" y1="38.1" x2="78.74" y2="15.24" width="0.1524" layer="91"/>
-<pinref part="SG1" gate="G$1" pin="1"/>
 </segment>
 </net>
 <net name="N$18" class="0">
 <segment>
+<pinref part="SG1" gate="G$1" pin="2"/>
 <pinref part="U$1" gate="G$1" pin="GND2"/>
 <wire x1="83.82" y1="38.1" x2="83.82" y2="25.4" width="0.1524" layer="91"/>
 <wire x1="83.82" y1="25.4" x2="71.12" y2="25.4" width="0.1524" layer="91"/>
-<pinref part="SG1" gate="G$1" pin="2"/>
 <wire x1="71.12" y1="25.4" x2="71.12" y2="15.24" width="0.1524" layer="91"/>
-</segment>
-</net>
+<junction x="71.12" y="15.24"/>
+<pinref part="LED1" gate="G$1" pin="C"/>
+<wire x1="55.88" y1="30.48" x2="55.88" y2="15.24" width="0.1524" layer="91"/>
+<wire x1="55.88" y1="15.24" x2="71.12" y2="15.24" width="0.1524" layer="91"/>
+</segment>
+</net>

Commit message: Plosne spoje
Connections:
- removed net N$18: LED1.C, SG1.2, U$1.GND2
- removed net N$6: C1.2, C2.2, NAPAJENI.1, R3.1, S1.P, S2.P1, U$1.GND, U$2.GND
- new net GND: C1.2, C2.2, LED1.C, NAPAJENI.1, R3.1, S1.P, S2.P1, SG1.2, U$1.GND, U$1.GND2, U$2.GND

Commit message: Finalni verze
Parts:
- removed MERENI_UBYTKU_NAPETI: (no value), pinhead:PINHD-1X2
- removed R4: 10, rcl:R-EU_0207/10
- added JP1, JP2: (no value), pinhead:PINHD-1X3
- added Q1, Q2: IRF4905, transistor-power:IRF4905
- added R10, R9: 2k, rcl:R-EU_0207/10
- R2, R5, R6, R7: value 10k -> 2k
Connections:
- removed net N$10: MERENI_UBYTKU_NAPETI.1, NAPAJENI.2, R4.2
- removed net N$8: U$1.GND1, UARTMODE.1
- new net N$18: JP1.3, Q1.D, Q2.D, R9.1, U$1.IO16
- new net N$19: JP1.2, U$1.EN
- new net N$20: JP1.1, R10.2
- new net N$6: C2.1, JP2.1, Q1.S, Q2.S, R1.2, R10.1, R2.2, R5.1, R6.1, R7.1, U$1.3.3V, U$2.OUT
- net GND: now also R9.2, S2.P, U$1.GND1, UARTMODE.1
- net N$1: now also JP2.3; no longer MERENI_UBYTKU_NAPETI.2, R4.1
- net N$12: now also Q2.G
- net N$13: now also Q1.G
- net N$2: now also JP2.2, NAPAJENI.2; no longer C2.1, R1.2, R2.2, R5.1, R6.1, R7.1, U$1.3.3V, U$1.EN, U$2.OUT
Other:
- moved on the sheet: D1, D2, R5, R6, R7, S1, S2
